Commit message: add launch

File: urdf/swerve.xacro (robot description, xacro)
@@ -18,5 +18,5 @@
     <origin xyz="0 0 0" rpy="0 0 0"/>
     <geometry>
-      <mesh filename="package://rere_daisha_ros/meshes/base_link.stl" scale="0.001 0.001 0.001"/>
+      <mesh filename="package://rere_daisha_ros/meshes/base_link.stl" scale="1 1 1"/>
     </geometry>
     <material name="_"/>
@@ -25,5 +25,5 @@
     <origin xyz="0 0 0" rpy="0 0 0"/>
     <geometry>
-      <mesh filename="package://rere_daisha_ros/meshes/base_link.stl" scale="0.001 0.001 0.001"/>
+      <mesh filename="package://rere_daisha_ros/meshes/base_link.stl" scale="1 1 1"/>
     </geometry>
   </collision>

Commit message: update 3Dlidar

File: urdf/swerve.xacro (robot description, xacro)
@@ -38,5 +38,5 @@
     <origin xyz="0.27 -0.155885 -0.015" rpy="0 0 0"/>
     <geometry>
-      <mesh filename="package://rere_daisha_ros/meshes/swerve_stare_v3_1.stl" scale="0.001 0.001 0.001"/>
+      <mesh filename="package://rere_daisha_ros/meshes/swerve_stare_v3_1.stl" scale="1 1 1"/>
     </geometry>
     <material name="_"/>
@@ -45,5 +45,5 @@
     <origin xyz="0.27 -0.155885 -0.015" rpy="0 0 0"/>
     <geometry>
-      <mesh filename="package://rere_daisha_ros/meshes/swerve_stare_v3_1.stl" scale="0.001 0.001 0.001"/>
+      <mesh filename="package://rere_daisha_ros/meshes/swerve_stare_v3_1.stl" scale="1 1 1"/>
     </geometry>
   </collision>
@@ -58,5 +58,5 @@
     <origin xyz="-0.27 -0.155885 -0.015" rpy="0 0 0"/>
     <geometry>
-      <mesh filename="package://rere_daisha_ros/meshes/swerve_stare_v3_2.stl" scale="0.001 0.001 0.001"/>
+      <mesh filename="package://rere_daisha_ros/meshes/swerve_stare_v3_2.stl" scale="1 1 1"/>
     </geometry>
     <material name="_"/>
@@ -65,5 +65,5 @@
     <origin xyz="-0.27 -0.155885 -0.015" rpy="0 0 0"/>
     <geometry>
-      <mesh filename="package://rere_daisha_ros/meshes/swerve_stare_v3_2.stl" scale="0.001 0.001 0.001"/>
+      <mesh filename="package://rere_daisha_ros/meshes/swerve_stare_v3_2.stl" scale="1 1 1"/>
     </geometry>
   </collision>
@@ -78,5 +78,5 @@
     <origin xyz="-0.0 0.311769 -0.015" rpy="0 0 0"/>
     <geometry>
-      <mesh filename="package://rere_daisha_ros/meshes/swerve_stare_v3_3.stl" scale="0.001 0.001 0.001"/>
+      <mesh filename="package://rere_daisha_ros/meshes/swerve_stare_v3_3.stl" scale="1 1 1"/>
     </geometry>
     <material name="_"/>
@@ -85,5 +85,5 @@
     <origin xyz="-0.0 0.311769 -0.015" rpy="0 0 0"/>
     <geometry>
-      <mesh filename="package://rere_daisha_ros/meshes/swerve_stare_v3_3.stl" scale="0.001 0.001 0.001"/>
+      <mesh filename="package://rere_daisha_ros/meshes/swerve_stare_v3_3.stl" scale="1 1 1"/>
     </geometry>
   </collision>
@@ -98,5 +98,5 @@
     <origin xyz="0.27 -0.155885 -0.005" rpy="0 0 0"/>
     <geometry>
-      <mesh filename="package://rere_daisha_ros/meshes/swerve_wheel_v4_1.stl" scale="0.001 0.001 0.001"/>
+      <mesh filename="package://rere_daisha_ros/meshes/swerve_wheel_v4_1.stl" scale="1 1 1"/>
     </geometry>
     <material name="_"/>
@@ -105,5 +105,5 @@
     <origin xyz="0.27 -0.155885 -0.005" rpy="0 0 0"/>
     <geometry>
-      <mesh filename="package://rere_daisha_ros/meshes/swerve_wheel_v4_1.stl" scale="0.001 0.001 0.001"/>
+      <mesh filename="package://rere_daisha_ros/meshes/swerve_wheel_v4_1.stl" scale="1 1 1"/>
     </geometry>
   </collision>
@@ -118,5 +118,5 @@
     <origin xyz="-0.27 -0.155885 -0.005" rpy="0 0 0"/>
     <geometry>
-      <mesh filename="package://rere_daisha_ros/meshes/swerve_wheel_v4_2.stl" scale="0.001 0.001 0.001"/>
+      <mesh filename="package://rere_daisha_ros/meshes/swerve_wheel_v4_2.stl" scale="1 1 1"/>
     </geometry>
     <material name="_"/>
@@ -125,5 +125,5 @@
     <origin xyz="-0.27 -0.155885 -0.005" rpy="0 0 0"/>
     <geometry>
-      <mesh filename="package://rere_daisha_ros/meshes/swerve_wheel_v4_2.stl" scale="0.001 0.001 0.001"/>
+      <mesh filename="package://rere_daisha_ros/meshes/swerve_wheel_v4_2.stl" scale="1 1 1"/>
     </geometry>
   </collision>
@@ -138,5 +138,5 @@
     <origin xyz="-0.0 0.311769 -0.005" rpy="0 0 0"/>
     <geometry>
-      <mesh filename="package://rere_daisha_ros/meshes/swerve_wheel_v4_3.stl" scale="0.001 0.001 0.001"/>
+      <mesh filename="package://rere_daisha_ros/meshes/swerve_wheel_v4_3.stl" scale="1 1 1"/>
     </geometry>
     <material name="_"/>
@@ -145,5 +145,5 @@
     <origin xyz="-0.0 0.311769 -0.005" rpy="0 0 0"/>
     <geometry>
-      <mesh filename="package://rere_daisha_ros/meshes/swerve_wheel_v4_3.stl" scale="0.001 0.001 0.001"/>
+      <mesh filename="package://rere_daisha_ros/meshes/swerve_wheel_v4_3.stl" scale="1 1 1"/>
     </geometry>
   </collision>
@@ -188,3 +188,52 @@
   <axis xyz="0.0 1.0 0.0"/>
 </joint>
+  <gazebo reference="base_link">
+    <sensor type="gpu_lidar" name="lidar_sensor">
+      <ignition_frame_id>base_link</ignition_frame_id>
+      <topic>/ldlidar_node/scan</topic>
+      <alwaysOn>1</alwaysOn>
+      <visualize>true</visualize>
+      <update_rate>10</update_rate>
+      <ray>
+        <scan>
+          <horizontal>
+            <samples>360</samples>
+            <resolution>1.0</resolution>
+            <min_angle>-1.3</min_angle>
+            <max_angle> 1.3</max_angle>
+          </horizontal>
+          <vertical>
+            <samples>1</samples>
+            <resolution>0.1</resolution>
+            <min_angle>-0.1221730476396</min_angle>
+            <max_angle>0.90757121103706</max_angle>
+          </vertical>
+        </scan>
+        <range>
+          <min>0.1</min>
+          <max>40.0</max>
+          <resolution>0.015</resolution>
+        </range>
+      </ray>
+      <plugin filename="libignition-gazebo-sensors-system.so" name="ignition::gazebo::systems::Sensors">
+          <render_engine>ogre</render_engine>
+      </plugin>
+    </sensor>
+  </gazebo>
+  <gazebo>
+    <plugin filename="libignition-gazebo-velocity-control-system.so"
+            name="ignition::gazebo::systems::VelocityControl">
+      <topic>/cmd_vel</topic>
+    </plugin>
+    <plugin filename="libignition-gazebo-odometry-publisher-system.so"
+          name="ignition::gazebo::systems::OdometryPublisher">
+    <odom_frame>odom</odom_frame>
+    <robot_base_frame>base_link</robot_base_frame>
+    <odom_publish_frequency>10</odom_publish_frequency>
+    <odom_topic>/odom</odom_topic>
+    <tf_topic>/tf</tf_topic>
+    <dimensions>2</dimensions>
+    <gaussian_noise>0.0</gaussian_noise>
+    </plugin>
+  </gazebo>
 </robot>

Commit message: add 3D LiDAR

File: urdf/swerve.xacro (robot description, xacro)
@@ -11,7 +11,7 @@
 <link name="base_link">
   <inertial>
-    <origin xyz="-5.775445040807947e-17 -0.021342710039809813 0.022104717930795586" rpy="0 0 0"/>
-    <mass value="6.8029685745384665"/>
-    <inertia ixx="0.146579" iyy="0.111575" izz="0.252635" ixy="0.0" iyz="0.002211" ixz="0.0"/>
+    <origin xyz="-9.205548913166534e-15 -0.021970869583044377 0.021991177325316028" rpy="0 0 0"/>
+    <mass value="6.743592473385616"/>
+    <inertia ixx="0.146238" iyy="0.111539" izz="0.252327" ixy="0.0" iyz="0.002266" ixz="0.0"/>
   </inertial>
   <visual>
@@ -146,4 +146,24 @@
     <geometry>
       <mesh filename="package://rere_daisha_ros/meshes/swerve_wheel_v4_3.stl" scale="1 1 1"/>
+    </geometry>
+  </collision>
+</link>
+<link name="mid-360-asm_v3_1">
+  <inertial>
+    <origin xyz="-0.001104909225108346 -1.70411760137823e-05 0.03018469043134761" rpy="0 0 0"/>
+    <mass value="0.4113191807928639"/>
+    <inertia ixx="0.000237" iyy="0.000251" izz="0.000164" ixy="-0.0" iyz="-0.0" ixz="-7e-06"/>
+  </inertial>
+  <visual>
+    <origin xyz="-0.0 -0.05 -0.07" rpy="0 0 0"/>
+    <geometry>
+      <mesh filename="package://rere_daisha_ros/meshes/mid-360-asm_v3_1.stl" scale="1 1 1"/>
+    </geometry>
+    <material name="_"/>
+  </visual>
+  <collision>
+    <origin xyz="-0.0 -0.05 -0.07" rpy="0 0 0"/>
+    <geometry>
+      <mesh filename="package://rere_daisha_ros/meshes/mid-360-asm_v3_1.stl" scale="1 1 1"/>
     </geometry>
   </collision>
@@ -187,4 +207,9 @@
   <child link="swerve_wheel_v4_3"/>
   <axis xyz="0.0 1.0 0.0"/>
+</joint>
+<joint name="rigit8" type="fixed">
+  <origin xyz="0.0 0.05 0.07" rpy="0 0 0"/>
+  <parent link="base_link"/>
+  <child link="mid-360-asm_v3_1"/>
 </joint>
 <gazebo reference="base_link">
