Commit message: update

File: urdf/materials.xacro (robot description, xacro)
@@ -7,3 +7,12 @@
   <color rgba="0.9607843137254902 0.9607843137254902 0.9647058823529412 1.0"/>
 </material>
+<material name="opaque160160160">
+  <color rgba="0.6274509803921569 0.6274509803921569 0.6274509803921569 1.0"/>
+</material>
+<material name="abs">
+  <color rgba="0.9647058823529412 0.9647058823529412 0.9529411764705882 1.0"/>
+</material>
+<material name="opaque252525">
+  <color rgba="0.09803921568627451 0.09803921568627451 0.09803921568627451 1.0"/>
+</material>
 </robot>

File: urdf/swerve.xacro (robot description, xacro)
@@ -253,4 +253,20 @@
   <d_gain>0.01</d_gain>
 </plugin>
+<plugin filename="gz-sim-joint-position-controller-system"
+        name="gz::sim::systems::JointPositionController">
+  <joint_name>swerve2</joint_name>
+  <topic>/pos_2</topic>
+  <p_gain>1</p_gain>
+  <i_gain>0.1</i_gain>
+  <d_gain>0.01</d_gain>
+</plugin>
+<plugin filename="gz-sim-joint-position-controller-system"
+        name="gz::sim::systems::JointPositionController">
+  <joint_name>swerve3</joint_name>
+  <topic>/pos_3</topic>
+  <p_gain>1</p_gain>
+  <i_gain>0.1</i_gain>
+  <d_gain>0.01</d_gain>
+</plugin>
 </gazebo>
 </robot>
