Commit message: change urdf

File: urdf/utan_urdf.xacro (robot description, xacro)
@@ -3,4 +3,10 @@
 <xacro:include filename="$(find utan_urdf_description)/urdf/materials.xacro" />
 <xacro:include filename="$(find utan_urdf_description)/urdf/utan_urdf.trans" />
+<link name="base_root"/>
+<joint name="base_root_to_base_link" type="fixed">
+  <origin xyz="0 0 0" rpy="0 0 0"/>
+  <parent link="base_root"/>
+  <child link="base_link"/>
+</joint>
 <link name="base_link">
   <inertial>

Commit message: update sim

File: urdf/utan_urdf.xacro (robot description, xacro)
@@ -1,6 +1,6 @@
 <?xml version="1.0" ?>
 <robot name="utan_urdf" xmlns:xacro="http://www.ros.org/wiki/xacro">
-<xacro:include filename="$(find utan_urdf_description)/urdf/materials.xacro" />
-<xacro:include filename="$(find utan_urdf_description)/urdf/utan_urdf.trans" />
+<xacro:include filename="$(find rere_daisha_ros)/urdf/materials.xacro" />
+<xacro:include filename="$(find rere_daisha_ros)/urdf/utan_urdf.trans" />
 <link name="base_root"/>
 <joint name="base_root_to_base_link" type="fixed">
@@ -18,5 +18,5 @@
     <origin xyz="0 0 0" rpy="0 0 0"/>
     <geometry>
-      <mesh filename="package://utan_urdf_description/meshes/base_link_utan.stl" scale="0.001 0.001 0.001"/>
+      <mesh filename="package://rere_daisha_ros/meshes/base_link_utan.stl" scale="0.001 0.001 0.001"/>
     </geometry>
     <material name="opaque160160160"/>
@@ -25,5 +25,5 @@
     <origin xyz="0 0 0" rpy="0 0 0"/>
     <geometry>
-      <mesh filename="package://utan_urdf_description/meshes/base_link_utan.stl" scale="0.001 0.001 0.001"/>
+      <mesh filename="package://rere_daisha_ros/meshes/base_link_utan.stl" scale="0.001 0.001 0.001"/>
     </geometry>
   </collision>
@@ -38,5 +38,5 @@
     <origin xyz="-0.11 -0.0 -0.08" rpy="0 0 0"/>
     <geometry>
-      <mesh filename="package://utan_urdf_description/meshes/turn_table_v2_1.stl" scale="0.001 0.001 0.001"/>
+      <mesh filename="package://rere_daisha_ros/meshes/turn_table_v2_1.stl" scale="0.001 0.001 0.001"/>
     </geometry>
     <material name="opaque160160160"/>
@@ -45,5 +45,5 @@
     <origin xyz="-0.11 -0.0 -0.08" rpy="0 0 0"/>
     <geometry>
-      <mesh filename="package://utan_urdf_description/meshes/turn_table_v2_1.stl" scale="0.001 0.001 0.001"/>
+      <mesh filename="package://rere_daisha_ros/meshes/turn_table_v2_1.stl" scale="0.001 0.001 0.001"/>
     </geometry>
   </collision>
@@ -58,5 +58,5 @@
     <origin xyz="-0.19163 -0.0 -0.0855" rpy="0 0 0"/>
     <geometry>
-      <mesh filename="package://utan_urdf_description/meshes/arm_frame_v2_1.stl" scale="0.001 0.001 0.001"/>
+      <mesh filename="package://rere_daisha_ros/meshes/arm_frame_v2_1.stl" scale="0.001 0.001 0.001"/>
     </geometry>
     <material name="abs"/>
@@ -65,5 +65,5 @@
     <origin xyz="-0.19163 -0.0 -0.0855" rpy="0 0 0"/>
     <geometry>
-      <mesh filename="package://utan_urdf_description/meshes/arm_frame_v2_1.stl" scale="0.001 0.001 0.001"/>
+      <mesh filename="package://rere_daisha_ros/meshes/arm_frame_v2_1.stl" scale="0.001 0.001 0.001"/>
     </geometry>
   </collision>
@@ -78,5 +78,5 @@
     <origin xyz="-0.0675 0.12025 -0.012" rpy="0 0 0"/>
     <geometry>
-      <mesh filename="package://utan_urdf_description/meshes/wheel_v1_1.stl" scale="0.001 0.001 0.001"/>
+      <mesh filename="package://rere_daisha_ros/meshes/wheel_v1_1.stl" scale="0.001 0.001 0.001"/>
     </geometry>
     <material name="opaque252525"/>
@@ -85,5 +85,5 @@
     <origin xyz="-0.0675 0.12025 -0.012" rpy="0 0 0"/>
     <geometry>
-      <mesh filename="package://utan_urdf_description/meshes/wheel_v1_1.stl" scale="0.001 0.001 0.001"/>
+      <mesh filename="package://rere_daisha_ros/meshes/wheel_v1_1.stl" scale="0.001 0.001 0.001"/>
     </geometry>
   </collision>
@@ -98,5 +98,5 @@
     <origin xyz="-0.0675 -0.12025 -0.012" rpy="0 0 0"/>
     <geometry>
-      <mesh filename="package://utan_urdf_description/meshes/wheel_v1_2.stl" scale="0.001 0.001 0.001"/>
+      <mesh filename="package://rere_daisha_ros/meshes/wheel_v1_2.stl" scale="0.001 0.001 0.001"/>
     </geometry>
     <material name="opaque252525"/>
@@ -105,5 +105,5 @@
     <origin xyz="-0.0675 -0.12025 -0.012" rpy="0 0 0"/>
     <geometry>
-      <mesh filename="package://utan_urdf_description/meshes/wheel_v1_2.stl" scale="0.001 0.001 0.001"/>
+      <mesh filename="package://rere_daisha_ros/meshes/wheel_v1_2.stl" scale="0.001 0.001 0.001"/>
     </geometry>
   </collision>
@@ -118,5 +118,5 @@
     <origin xyz="-0.279945 0.0 -0.019" rpy="0 0 0"/>
     <geometry>
-      <mesh filename="package://utan_urdf_description/meshes/ldlidar_v1_1.stl" scale="0.001 0.001 0.001"/>
+      <mesh filename="package://rere_daisha_ros/meshes/ldlidar_v1_1.stl" scale="0.001 0.001 0.001"/>
     </geometry>
     <material name="_"/>
@@ -125,5 +125,5 @@
     <origin xyz="-0.279945 0.0 -0.019" rpy="0 0 0"/>
     <geometry>
-      <mesh filename="package://utan_urdf_description/meshes/ldlidar_v1_1.stl" scale="0.001 0.001 0.001"/>
+      <mesh filename="package://rere_daisha_ros/meshes/ldlidar_v1_1.stl" scale="0.001 0.001 0.001"/>
     </geometry>
   </collision>
@@ -138,5 +138,5 @@
     <origin xyz="-0.27463 -0.0175 -0.11" rpy="0 0 0"/>
     <geometry>
-      <mesh filename="package://utan_urdf_description/meshes/vertical_arm_frame_v2_1.stl" scale="0.001 0.001 0.001"/>
+      <mesh filename="package://rere_daisha_ros/meshes/vertical_arm_frame_v2_1.stl" scale="0.001 0.001 0.001"/>
     </geometry>
     <material name="_"/>
@@ -145,5 +145,5 @@
     <origin xyz="-0.27463 -0.0175 -0.11" rpy="0 0 0"/>
     <geometry>
-      <mesh filename="package://utan_urdf_description/meshes/vertical_arm_frame_v2_1.stl" scale="0.001 0.001 0.001"/>
+      <mesh filename="package://rere_daisha_ros/meshes/vertical_arm_frame_v2_1.stl" scale="0.001 0.001 0.001"/>
     </geometry>
   </collision>
@@ -158,5 +158,5 @@
     <origin xyz="-0.35963 0.0075 -0.2" rpy="0 0 0"/>
     <geometry>
-      <mesh filename="package://utan_urdf_description/meshes/arm_edge_v2_1.stl" scale="0.001 0.001 0.001"/>
+      <mesh filename="package://rere_daisha_ros/meshes/arm_edge_v2_1.stl" scale="0.001 0.001 0.001"/>
     </geometry>
     <material name="opaque160160160"/>
@@ -165,5 +165,5 @@
     <origin xyz="-0.35963 0.0075 -0.2" rpy="0 0 0"/>
     <geometry>
-      <mesh filename="package://utan_urdf_description/meshes/arm_edge_v2_1.stl" scale="0.001 0.001 0.001"/>
+      <mesh filename="package://rere_daisha_ros/meshes/arm_edge_v2_1.stl" scale="0.001 0.001 0.001"/>
     </geometry>
   </collision>
@@ -178,5 +178,5 @@
     <origin xyz="-0.23463 -0.0275 -0.41" rpy="0 0 0"/>
     <geometry>
-      <mesh filename="package://utan_urdf_description/meshes/utan_figure_v2_1.stl" scale="0.001 0.001 0.001"/>
+      <mesh filename="package://rere_daisha_ros/meshes/utan_figure_v2_1.stl" scale="0.001 0.001 0.001"/>
     </geometry>
     <material name="abs"/>
@@ -185,5 +185,5 @@
     <origin xyz="-0.23463 -0.0275 -0.41" rpy="0 0 0"/>
     <geometry>
-      <mesh filename="package://utan_urdf_description/meshes/utan_figure_v2_1.stl" scale="0.001 0.001 0.001"/>
+      <mesh filename="package://rere_daisha_ros/meshes/utan_figure_v2_1.stl" scale="0.001 0.001 0.001"/>
     </geometry>
   </collision>
@@ -223,5 +223,5 @@
   <child link="vertical_arm_frame_v2_1"/>
   <axis xyz="0.0 -0.0 1.0"/>
-  <limit upper="0.0" lower="0.17" effort="100" velocity="100"/>
+  <limit upper="0.17" lower="0.0" effort="100" velocity="100"/>
 </joint>
 <joint name="arm_horizontal" type="prismatic">
@@ -230,5 +230,5 @@
   <child link="arm_edge_v2_1"/>
   <axis xyz="1.0 0.0 -0.0"/>
-  <limit upper="0.0" lower="0.085" effort="100" velocity="100"/>
+  <limit upper="0.085" lower="0.0" effort="100" velocity="100"/>
 </joint>
 <joint name="utan" type="fixed">

Commit message: change mesh

File: urdf/utan_urdf.xacro (robot description, xacro)
@@ -83,7 +83,7 @@
   </visual>
   <collision>
-    <origin xyz="-0.0675 0.12025 -0.012" rpy="0 0 0"/>
-    <geometry>
-      <mesh filename="package://rere_daisha_ros/meshes/wheel_v1_1.stl" scale="0.001 0.001 0.001"/>
+    <origin xyz="0 0.0177 0" rpy="1.57 0 0"/>
+    <geometry>
+      <cylinder radius="0.032" length="0.0354"/>
     </geometry>
   </collision>
@@ -103,7 +103,7 @@
   </visual>
   <collision>
-    <origin xyz="-0.0675 -0.12025 -0.012" rpy="0 0 0"/>
-    <geometry>
-      <mesh filename="package://rere_daisha_ros/meshes/wheel_v1_2.stl" scale="0.001 0.001 0.001"/>
+    <origin xyz="0 -0.0177 0" rpy="1.57 0 0"/>
+    <geometry>
+      <cylinder radius="0.032" length="0.0354"/>
     </geometry>
   </collision>
@@ -276,4 +276,5 @@
   <topic>/wheel_right</topic>
   <initial_velocity>0</initial_velocity>
+  <!-- <use_force_commands>true</use_force_commands> -->
   <p_gain>1</p_gain>
   <i_gain>0.1</i_gain>
@@ -285,4 +286,5 @@
   <topic>/wheel_left</topic>
   <initial_velocity>0</initial_velocity>
+  <!-- <use_force_commands>true</use_force_commands> -->
   <p_gain>1</p_gain>
   <i_gain>0.1</i_gain>

Commit message: add diff drive

File: urdf/utan_urdf.xacro (robot description, xacro)
@@ -211,5 +211,5 @@
   <parent link="base_link"/>
   <child link="wheel_v1_2"/>
-  <axis xyz="0.0 -1.0 0.0"/>
+  <axis xyz="0.0 1.0 0.0"/>
 </joint>
 <joint name="lidar_joint" type="fixed">
@@ -271,24 +271,13 @@
 <!-- wheel -->
 <gazebo>
-<plugin filename="gz-sim-joint-controller-system"
-        name="gz::sim::systems::JointController">
-  <joint_name>wheel_right</joint_name>
-  <topic>/wheel_right</topic>
-  <initial_velocity>0</initial_velocity>
-  <!-- <use_force_commands>true</use_force_commands> -->
-  <p_gain>1</p_gain>
-  <i_gain>0.1</i_gain>
-  <d_gain>0.01</d_gain>
-</plugin>
-<plugin filename="gz-sim-joint-controller-system"
-        name="gz::sim::systems::JointController">
-  <joint_name>wheel_left</joint_name>
-  <topic>/wheel_left</topic>
-  <initial_velocity>0</initial_velocity>
-  <!-- <use_force_commands>true</use_force_commands> -->
-  <p_gain>1</p_gain>
-  <i_gain>0.1</i_gain>
-  <d_gain>0.01</d_gain>
-</plugin>
+  <plugin filename="gz-sim-diff-drive-system"
+          name="gz::sim::systems::DiffDrive">
+    <left_joint>wheel_left</left_joint>
+    <right_joint>wheel_right</right_joint>
+    <wheel_separation>0.2405</wheel_separation>
+    <wheel_radius>0.0321</wheel_radius>
+    <topic>cmd_vel</topic>
+    <odom_publish_frequency>50</odom_publish_frequency>
+  </plugin>
 </gazebo>
 <!-- arm -->
@@ -312,3 +301,7 @@
   <mu2>1.0</mu2>
 </gazebo>
+<gazebo reference="base_link">
+  <mu1>0</mu1>
+  <mu2>0</mu2>
+</gazebo>
 </robot>

Commit message: update urdf

File: urdf/utan_urdf.xacro (robot description, xacro)
@@ -219,9 +219,9 @@
 </joint>
 <joint name="arm_vertical" type="prismatic">
-  <origin xyz="0.083 0.0175 0.0245" rpy="0 0 0"/>
+  <origin xyz="0.083 0.015 0.0245" rpy="0 0 0"/>
   <parent link="arm_frame_v2_1"/>
   <child link="vertical_arm_frame_v2_1"/>
   <axis xyz="0.0 -0.0 1.0"/>
-  <limit upper="0.17" lower="0.0" effort="100" velocity="100"/>
+  <limit upper="0.17" lower="-0.02" effort="1000" velocity="100"/>
 </joint>
 <joint name="arm_horizontal" type="prismatic">
@@ -287,7 +287,7 @@
   <joint_name>arm_yaw</joint_name>
   <topic>/arm_yaw</topic>
-  <p_gain>20</p_gain>
+  <p_gain>2</p_gain>
   <i_gain>0.1</i_gain>
-  <d_gain>0.01</d_gain>
+  <d_gain>1</d_gain>
 </plugin>
 <plugin filename="gz-sim-joint-position-controller-system"
@@ -298,4 +298,6 @@
   <i_gain>0.5</i_gain>
   <d_gain>0.01</d_gain>
+  <use_velocity_commands>true</use_velocity_commands>
+  <cmd_max>0.5</cmd_max>
 </plugin>
 <plugin filename="gz-sim-joint-position-controller-system"
@@ -303,7 +305,7 @@
   <joint_name>arm_horizontal</joint_name>
   <topic>/arm_horizontal</topic>
-  <p_gain>10</p_gain>
+  <p_gain>2</p_gain>
   <i_gain>0.5</i_gain>
-  <d_gain>0.01</d_gain>
+  <d_gain>1</d_gain>
 </plugin>
 </gazebo>

Commit message: add caster

File: urdf/utan_urdf.xacro (robot description, xacro)
@@ -189,4 +189,22 @@
   </collision>
 </link>
+<link name="caster_ball">
+  <inertial>
+    <mass value="0.05"/>
+    <inertia ixx="1e-5" iyy="1e-5" izz="1e-5" ixy="0" ixz="0" iyz="0"/>
+  </inertial>
+  <collision>
+    <origin xyz="0 0 0" rpy="0 0 0"/>
+    <geometry>
+      <sphere radius="0.015"/>
+    </geometry>
+  </collision>
+  <visual>
+    <origin xyz="0 0 0" rpy="0 0 0"/>
+    <geometry>
+      <sphere radius="0.015"/>
+    </geometry>
+  </visual>
+</link>
 <joint name="rigit1" type="fixed">
   <origin xyz="0.11 0.0 0.08" rpy="0 0 0"/>
@@ -236,4 +254,10 @@
   <parent link="arm_frame_v2_1"/>
   <child link="utan_figure_v2_1"/>
+</joint>
+<joint name="caster_ball_joint" type="fixed">
+  <!-- ここは「地面に接する高さ」になるよう調整 -->
+  <origin xyz="0.235484 0 -0.006" rpy="0 0 0"/>
+  <parent link="base_link"/>
+  <child link="caster_ball"/>
 </joint>
 <gazebo reference="ldlidar_v1_1">
@@ -320,6 +344,10 @@
 </gazebo>
 <gazebo reference="base_link">
-  <mu1>0</mu1>
-  <mu2>0</mu2>
+  <mu1>1.0</mu1>
+  <mu2>1.0</mu2>
+</gazebo>
+<gazebo reference="caster_ball">
+  <mu1>0.3</mu1>
+  <mu2>0.3</mu2>
 </gazebo>
 </robot>

Commit message: update joint

File: urdf/utan_urdf.xacro (robot description, xacro)
@@ -207,4 +207,6 @@
   </visual>
 </link>
+<link name="lidar_link">
+</link>
 <joint name="rigit1" type="fixed">
   <origin xyz="0.11 0.0 0.08" rpy="0 0 0"/>
@@ -255,18 +257,22 @@
   <child link="utan_figure_v2_1"/>
 </joint>
+<joint name="lidar_joint_true" type="fixed">
+  <origin xyz="0.017 0 -0.0291" rpy="3.14159 0 0"/>
+  <parent link="ldlidar_v1_1"/>
+  <child link="lidar_link"/>
+</joint>
 <joint name="caster_ball_joint" type="fixed">
   <!-- ここは「地面に接する高さ」になるよう調整 -->
-  <origin xyz="0.235484 0 -0.006" rpy="0 0 0"/>
+  <origin xyz="0.235484 0 -0.005" rpy="0 0 0"/>
   <parent link="base_link"/>
   <child link="caster_ball"/>
 </joint>
-<gazebo reference="ldlidar_v1_1">
+<gazebo reference="lidar_link">
   <sensor type="gpu_lidar" name="lidar_sensor">
-    <ignition_frame_id>ldlidar_v1_1</ignition_frame_id>
+    <ignition_frame_id>lidar_link</ignition_frame_id>
     <topic>/ldlidar_node/scan</topic>
     <alwaysOn>1</alwaysOn>
     <visualize>true</visualize>
     <update_rate>10</update_rate>
-    <pose>0 0 -0.04 0 0 0</pose>
     <ray>
       <scan>
@@ -283,5 +289,5 @@
       </scan>
       <range>
-        <min>0.02</min>
+        <min>0.04</min>
         <max>12.0</max>
         <resolution>0.015</resolution>
